File: Proyecto/Kikad/Placa_Principal/Placa_Principal/Placa_Principal.kicad_pcb (KiCad board)
At the start: 2 copper layers, 9 parts, among them J1 Screw_Terminal_01x03, J2 Screw_Terminal_01x03, J3 Screw_Terminal_01x03, J4 Screw_Terminal_01x03, J5 USB_C_Receptacle_PowerOnly_6P, SW1 SW_DIP_x01, SW1 SW_Nidec_CAS-120A1, U1 ESP32-DEVKITC-32D

Commit message: Hice la Placa_Principal y corregi algunos detalles de la placa modulo rele
Parts:
- removed the SW1 at (135.8, 84.6)
- added G***: LOGO, Logo:Logo_Cobre_4.8mm_7mm, F.Cu at (217.8, 89.5)
- added G***: LOGO, Logo:Logo_Cobre_4.8mm_7mm, B.Cu at (217.9, 89.6)
- added J6: Screw_Terminal_01x07, Huellas:PinHeader_1x07_P2.54mm_Vertical, F.Cu at (202.2, 114.9)
- J4: footprint Connector_PinHeader_2.54mm:PinHeader_1x03_P2.54mm_Vertical -> Huellas:PinHeader_1x03_P2.54mm_Vertical
- SW1: footprint Button_Switch_THT:SW_DIP_SPSTx01_Slide_6.7x4.1mm_W7.62mm_P2.54mm_LowProfile -> Huellas:PinHeader_1x03_P2.54mm_Vertical
- moved J1 111.8 mm to (232.4, 36.2)
- moved J2 95.0 mm to (232.4, 57.1)
- moved C1 94.1 mm to (213.4, 97.1), turned to -90 degrees
- moved J3 90.4 mm to (232.4, 78.1)
- moved J5 82.2 mm to (195.0, 93.3), turned to -90 degrees
- moved J4 68.0 mm to (232.4, 99.1)
- moved SW1 24.8 mm to (193.0, 103.5), turned to 90 degrees
- moved U1 0.15 mm to (207.6, 56.4), turned to 180 degrees
Connections:
- C1 pad 1: +5V -> GND
- C1 pad 2: GND -> +5V
- J5 pad A9: +5V -> Net-(J5-VBUS-PadA9)
- J5 pad B9: +5V -> Net-(J5-VBUS-PadA9)
- SW1 pad 1: +5V -> Net-(J5-VBUS-PadA9)
- SW1 pad 2: Entrada_A -> +5V
- U1 pad P18: GPIO_12 -> GPIO_18
Routing:
- net +5V: track 0.00 -> 149.7 mm, vias 0 -> 5
- net GPIO_16: track 0.00 -> 67.9 mm
- net GPIO_17: track 0.00 -> 64.0 mm
- net GPIO_33: track 0.00 -> 61.3 mm
- net GPIO_18: track 0.00 -> 58.2 mm
- net GPIO_32: track 0.00 -> 55.9 mm
- net GPIO_25: track 0.00 -> 55.5 mm
- net GND: track 0.00 -> 55.1 mm
- net GPIO_26: track 0.00 -> 36.7 mm
- net GPIO_14: track 0.00 -> 21.3 mm
- net GPIO_27: track 0.00 -> 18.0 mm
- net Net-(J5-VBUS-PadA9): track 0.00 -> 16.8 mm
- net (no net): vias 0 -> 8
- added copper zone on B.Cu, net GND
- added copper zone on F.Cu, net GND
Other:
- board outline added: 43.8 x 87 mm

Commit message: Arregle unas cosas de las dos placas
Connections:
- C1 pad 2: +5V -> (no net)
- J1 pad 1: +5V -> (no net)
- J2 pad 1: +5V -> (no net)
- J3 pad 1: +5V -> (no net)
- J4 pad 1: +5V -> (no net)
- J6 pad 2: +5V -> (no net)
- SW1 pad 2: +5V -> (no net)
- U1 pad 5V: +5V -> (no net)
Routing:
- net +5V: track 149.7 -> 38.5 mm, vias 5 -> 0
- net (no net): track 0.00 -> 92.3 mm
- net GND: track 55.1 -> 36.1 mm
- net GPIO_14: track 21.3 -> 17.6 mm
- net GPIO_25: track 55.5 -> 52.6 mm
- net GPIO_26: track 36.7 -> 36.0 mm
Other:
- board size 43.8 x 87 mm -> 46.4 x 87 mm
