File: Proyecto/Kikad/Placa_Principal/Placa_Principal/Placa_Principal.kicad_pcb (KiCad board)
At the start: 2 copper layers, 46.4 x 87 mm, 11 parts, among them J1 Screw_Terminal_01x03, J2 Screw_Terminal_01x03, J3 Screw_Terminal_01x03, J4 Screw_Terminal_01x03, J5 USB_C_Receptacle_PowerOnly_6P, J6 Screw_Terminal_01x07, SW1 SW_DIP_x01, U1 ESP32-DEVKITC-32D

Commit message: Cambie 2 gpio
Connections:
- J6 pad 6: GPIO_17 -> GPIO_21
- J6 pad 7: GPIO_18 -> GPIO_22
- U1 pad P17: GPIO_17 -> unconnected-(U1-IO17-PadP17)
- U1 pad P18: GPIO_18 -> unconnected-(U1-IO18-PadP18)
- U1 pad P21: unconnected-(U1-IO21-PadP21) -> GPIO_21
- U1 pad P22: unconnected-(U1-IO22-PadP22) -> GPIO_22
Routing:
- net GPIO_17: track 64.0 -> 0.00 mm
- net GPIO_18: track 58.2 -> 0.00 mm
- net GPIO_21: track 0.00 -> 53.2 mm
- net GPIO_22: track 0.00 -> 43.4 mm
Changed lines of the file:
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@@
 	(net 1 "+5V")
 	(net 2 "Net-(J5-VBUS-PadA9)")
-	(net 3 "GPIO_18")
+	(net 3 "GPIO_21")
 	(net 4 "unconnected-(U1-IO5-PadP05)")
 	(net 5 "unconnected-(U1-PadGND1)")
@@
 	(net 9 "unconnected-(U1-PadEN)")
 	(net 10 "unconnected-(U1-IO19-PadP19)")
-	(net 11 "unconnected-(U1-IO22-PadP22)")
+	(net 11 "GPIO_22")
 	(net 12 "unconnected-(U1-PadSD3)")
 	(net 13 "unconnected-(U1-PadSD0)")
@@
 	(net 27 "unconnected-(U1-IO34-PadP34)")
 	(net 28 "unconnected-(U1-IO4-PadP04)")
-	(net 29 "unconnected-(U1-IO21-PadP21)")
+	(net 29 "unconnected-(U1-IO17-PadP17)")
 	(net 30 "unconnected-(U1-SENSOR_VN-PadSVN)")
 	(net 31 "unconnected-(J5-SHIELD-PadS1)")
@@
 	(net 33 "GND")
 	(net 34 "unconnected-(J5-CC2-PadB5)")
-	(net 35 "GPIO_17")
+	(net 35 "unconnected-(U1-IO18-PadP18)")
 	(net 36 "GPIO_32")
 	(net 37 "GPIO_16")
@@
 			(layers "*.Cu" "*.Mask")
 			(remove_unused_layers no)
-			(net 35 "GPIO_17")
+			(net 29 "unconnected-(U1-IO17-PadP17)")
 			(pinfunction "IO17")
 			(pintype "bidirectional")
@@
 			(layers "*.Cu" "*.Mask")
 			(remove_unused_layers no)
-			(net 3 "GPIO_18")
+			(net 35 "unconnected-(U1-IO18-PadP18)")
 			(pinfunction "IO18")
 			(pintype "bidirectional")
@@
 			(layers "*.Cu" "*.Mask")
 			(remove_unused_layers no)
-			(net 29 "unconnected-(U1-IO21-PadP21)")
+			(net 3 "GPIO_21")
 			(pinfunction "IO21")
 			(pintype "bidirectional")
@@
 			(layers "*.Cu" "*.Mask")
 			(remove_unused_layers no)
-			(net 11 "unconnected-(U1-IO22-PadP22)")
+			(net 11 "GPIO_22")
 			(pinfunction "IO22")
 			(pintype "bidirectional")
@@
 			(layers "*.Cu" "*.Mask")
 			(remove_unused_layers no)
-			(net 35 "GPIO_17")
+			(net 3 "GPIO_21")
 			(pinfunction "Pin_6")
 			(pintype "passive")
@@
 			(layers "*.Cu" "*.Mask")
 			(remove_unused_layers no)
-			(net 3 "GPIO_18")
+			(net 11 "GPIO_22")
 			(pinfunction "Pin_7")
 			(pintype "passive")
@@
 	)
 	(segment
-		(start 198.12 55.88)
-		(end 194.945 55.88)
+		(start 203.28 109.855)
+		(end 203.28 66.12)
 		(width 1)
 		(layer "B.Cu")
@@
 	)
 	(segment
-		(start 200.66 58.42)
-		(end 198.12 55.88)
+		(start 200.66 63.5)
+		(end 194.945 63.5)
 		(width 1)
 		(layer "B.Cu")
@@
 	)
 	(segment
-		(start 200.74 109.855)
-		(end 200.66 109.775)
+		(start 203.28 66.12)
+		(end 200.66 63.5)
 		(width 1)
 		(layer "B.Cu")
@@
 	)
 	(segment
+		(start 200.66 73.025)
+		(end 198.755 71.12)
+		(width 1)
+		(layer "B.Cu")
+		(net 11)
+	)
+	(segment
 		(start 200.66 109.775)
-		(end 200.66 58.42)
+		(end 200.66 73.025)
 		(width 1)
 		(layer "B.Cu")
-		(net 3)
+		(net 11)
+	)
+	(segment
+		(start 198.755 71.12)
+		(end 194.945 71.12)
+		(width 1)
+		(layer "B.Cu")
+		(net 11)
+	)
+	(segment
+		(start 200.74 109.855)
+		(end 200.66 109.775)
+		(width 1)
+		(layer "B.Cu")
+		(net 11)
 	)
 	(segment
@@
 	)
 	(segment
-		(start 203.28 109.855)
-		(end 203.28 56.595)
-		(width 1)
-		(layer "B.Cu")
-		(net 35)
-	)
-	(segment
-		(start 203.28 56.595)
-		(end 197.485 50.8)
-		(width 1)
-		(layer "B.Cu")
-		(net 35)
-	)
-	(segment
-		(start 197.485 50.8)
-		(end 194.945 50.8)
-		(width 1)
-		(layer "B.Cu")
-		(net 35)
-	)
-	(segment

Commit message: Cambie los gpio y agregue un exel
Connections:
- J1 pad 2: GPIO_13 -> GPIO_16
- J2 pad 2: GPIO_12 -> GPIO_17
- J3 pad 2: GPIO_27 -> GPIO_33
- J4 pad 2: GPIO_25 -> GPIO_32
- J6 pad 3: GPIO_32 -> GPIO_18
- J6 pad 4: GPIO_33 -> GPIO_19
- J6 pad 5: GPIO_16 -> GPIO_21
- J6 pad 6: GPIO_21 -> GPIO_22
- J6 pad 7: GPIO_22 -> GPIO_23
- U1 pad P12: GPIO_12 -> unconnected-(U1-IO12-PadP12)
- U1 pad P13: GPIO_13 -> (no net)
- U1 pad P14: unconnected-(U1-IO14-PadP14) -> (no net)
- U1 pad P17: unconnected-(U1-IO17-PadP17) -> GPIO_17
- U1 pad P18: unconnected-(U1-IO18-PadP18) -> GPIO_18
- U1 pad P19: unconnected-(U1-IO19-PadP19) -> GPIO_19
- U1 pad P23: unconnected-(U1-IO23-PadP23) -> GPIO_23
- U1 pad P25: GPIO_25 -> unconnected-(U1-IO25-PadP25)
- U1 pad P26: unconnected-(U1-IO26-PadP26) -> (no net)
- U1 pad P27: GPIO_27 -> (no net)
- U1 pad SD2: unconnected-(U1-PadSD2) -> (no net)
- U1 pad SD3: unconnected-(U1-PadSD3) -> (no net)
Routing:
- net GPIO_18: track 0.00 -> 67.9 mm
- net GPIO_19: track 0.00 -> 62.9 mm
- net GPIO_25: track 52.6 -> 0.00 mm
- net GPIO_17: track 0.00 -> 41.1 mm
- net GPIO_23: track 0.00 -> 40.2 mm
- net +5V: track 130.8 -> 168.5 mm
- net GPIO_27: track 37.5 -> 0.00 mm
- net GPIO_33: track 61.3 -> 31.7 mm
- net GPIO_16: track 67.9 -> 44.0 mm
- net GPIO_12: track 22.4 -> 0.00 mm
- net GPIO_13: track 12.9 -> 0.00 mm
- net GPIO_32: track 55.9 -> 47.9 mm
- net GPIO_21: track 53.2 -> 55.3 mm
- net GPIO_22: track 43.4 -> 45.2 mm
